Commit message: camera

File: my_robot_gazebo/urdf/my_robot.urdf.xacro (robot description, xacro)
@@ -12,5 +12,5 @@
 	<link name ="base_link">
 		<collision>
-			<origin xyz ="0 0 1.2"/>
+			<origin xyz ="0 0 0.3"/>
 			<geometry>
 				<cylinder length = "0.6" radius = "1.85"/>
@@ -21,12 +21,13 @@
 				<cylinder length = "0.6" radius = "1.85"/>
 			</geometry>
-			<origin xyz ="0 0 1.2"/>
+			<origin xyz ="0 0 0.3"/>
 		</visual>
         <xacro:default_inertial mass = "0.5"/>
 	</link>
-	<joint name = "world_to_base" type= "fixed">
+	<joint name = "world_to_base" type= "continuous">
+		<axis xyz = "0 0 1"/>
 		<parent link = "world"/>
 		<child link = "base_link"/>
-		<origin xyz = "0 0 -0.9"/>
+		<origin xyz = "0 0 0"/>
 		<!--<dynamics damping="0.7"/>-->
 	</joint>
@@ -70,5 +71,5 @@
       	</inertial>
 	</link>
-	<joint name ="base_to_${name_leg}" type ="revolute">
+	<joint name ="base_to_${name_leg}" type ="fixed"> <!--revolute-->
 		<axis xyz="0 0 1"/>
 		<limit effort= "1000.0" lower="-1" upper="1" velocity="0.3"/>
@@ -97,5 +98,5 @@
       	</inertial>
 	</link>
-	<joint name = "${name_leg}_to_${number_wheel}" type = "continuous">
+	<joint name = "${name_leg}_to_${number_wheel}" type = "continuous"> <!--continuous-->
 		<axis xyz="0 1 0"/>
 		<limit effort= "1000.0" velocity="1"/>
@@ -105,4 +106,5 @@
 		<dynamics damping="0.5"/>
 	</joint>
+<!--
 	<transmission name="trainsmision_${name_leg}">
      	<type>transmission_interface/SimpleTransmission</type>
@@ -114,5 +116,5 @@
       		<mechanicalReduction>1</mechanicalReduction>
      	</actuator>
-  	</transmission>
+  	</transmission>-->
     <transmission name="transmission_${number_wheel}">
      	<type>transmission_interface/SimpleTransmission</type>
@@ -126,12 +128,51 @@
   	</transmission>
 </xacro:macro>
+<!--
+	<transmission name="trainsm_weel4">
+     	<type>transmission_interface/SimpleTransmission</type>
+     	<joint name="fourth_leg_to_wheel4">
+      		<hardwareInterface>hardware_interface/EffortJointInterface</hardwareInterface>
+     	</joint>
+     	<actuator name="motor_w4">
+      		<hardwareInterface>hardware_interface/EffortJointInterface</hardwareInterface>
+      		<mechanicalReduction>1</mechanicalReduction>
+     	</actuator>
+  	</transmission>-->
+<xacro:property name="camera_link" value="0.1" /> <!-- Size of square 'camera' box -->
+	<joint name="camera_joint" type="fixed">
+    	<axis xyz="0 1 0" />
+    	<origin xyz="0.25 0.4 0.25" rpy="0 0 1.71"/>
+    	<parent link="wheel4"/>
+    	<child link="camera_link"/>
+  	</joint>
+  	<!-- Camera -->
+  	<link name="camera_link">
+    	<collision>
+      		<origin xyz="0 0 0" rpy="0 0 0"/>
+      		<geometry>
+    			<box size="${camera_link} ${camera_link} ${camera_link}"/>
+      		</geometry>
+    	</collision>
+		<visual>
+      		<origin xyz="0 0 0" rpy="0 0 0"/>
+      		<geometry>
+    			<box size="${camera_link} ${camera_link} ${camera_link}"/>
+      		</geometry>
+      		<material name="red"/>
+    	</visual>
+    	<inertial>
+      		<mass value="1e-5" />
+      		<origin xyz="0 0 0" rpy="0 0 0"/>
+      		<inertia ixx="1e-6" ixy="0" ixz="0" iyy="1e-6" iyz="0" izz="1e-6" />
+    	</inertial>
+  	</link>
 <xacro:link_leg name_leg = "first_leg" number_wheel = "wheel1"
-	            coord_joint = "1 1 0.9" angles_joint = "0 0 0"/>
+	            coord_joint = "1 1 0" angles_joint = "0 0 0"/>
 <xacro:link_leg name_leg = "second_leg" number_wheel = "wheel2"
-	            coord_joint = "-1 -1 0.9" angles_joint = "0 0 3.142"/>
+	            coord_joint = "-1 -1 0" angles_joint = "0 0 3.142"/>
 <xacro:link_leg name_leg = "third_leg" number_wheel = "wheel3"
-	            coord_joint = "-1 1 0.9" angles_joint= "0 0 0"/>
+	            coord_joint = "-1 1 0" angles_joint= "0 0 0"/>
 <xacro:link_leg name_leg = "fourth_leg" number_wheel = "wheel4"
-	            coord_joint = "1 -1 0.9" angles_joint= "0 0 3.142"/>
+	            coord_joint = "1 -1 0" angles_joint= "0 0 3.142"/>
 <gazebo>
   <plugin name="gazebo_ros_control" filename="libgazebo_ros_control.so">
@@ -139,3 +180,43 @@
   </plugin>
 </gazebo>
+<!-- camera -->
+  <gazebo reference="camera_link">
+    <sensor type="camera" name="camera1">
+      <update_rate>30.0</update_rate>
+      <camera name="head">
+        <horizontal_fov>1.3962634</horizontal_fov>
+        <image>
+          <width>800</width>
+          <height>800</height>
+          <format>R8G8B8</format>
+        </image>
+        <clip>
+          <near>0.02</near>
+          <far>300</far>
+        </clip>
+        <noise>
+          <type>gaussian</type>
+          <!-- Noise is sampled independently per pixel on each frame.
+               That pixel's noise value is added to each of its color
+               channels, which at that point lie in the range [0,1]. -->
+          <mean>0.0</mean>
+          <stddev>0.007</stddev>
+        </noise>
+      </camera>
+      <plugin name="camera_controller" filename="libgazebo_ros_camera.so">
+        <alwaysOn>true</alwaysOn>
+        <updateRate>0.0</updateRate>
+        <cameraName>camrobot/camera1</cameraName>
+        <imageTopicName>image_raw</imageTopicName>
+        <cameraInfoTopicName>camera_info</cameraInfoTopicName>
+        <frameName>camera_link</frameName>
+        <hackBaseline>0.07</hackBaseline>
+        <distortionK1>0.0</distortionK1>
+        <distortionK2>0.0</distortionK2>
+        <distortionK3>0.0</distortionK3>
+        <distortionT1>0.0</distortionT1>
+        <distortionT2>0.0</distortionT2>
+      </plugin>
+    </sensor>
+  </gazebo>
 </robot>

Commit message: Fixing some conservation

File: my_robot_gazebo/urdf/my_robot.urdf.xacro (robot description, xacro)
@@ -1,4 +1,5 @@
 <?xml version="1.0" ?> <!--encoding="utf-8"-->
 <robot name ="my_robot" xmlns:xacro="http://www.ros.org/wiki/xacro" >
+<xacro:include filename="$(find my_robot_gazebo)/urdf/camera_on_wheel.xacro" />
 	<link name = "world"/>
 <xacro:macro name="default_inertial" params="mass">
@@ -25,5 +26,5 @@
         <xacro:default_inertial mass = "0.5"/>
 	</link>
-	<joint name = "world_to_base" type= "continuous">
+	<joint name = "world_to_base" type= "fixed">
 		<axis xyz = "0 0 1"/>
 		<parent link = "world"/>
@@ -128,43 +129,4 @@
   	</transmission>
 </xacro:macro>
-<!--
-	<transmission name="trainsm_weel4">
-     	<type>transmission_interface/SimpleTransmission</type>
-     	<joint name="fourth_leg_to_wheel4">
-      		<hardwareInterface>hardware_interface/EffortJointInterface</hardwareInterface>
-     	</joint>
-     	<actuator name="motor_w4">
-      		<hardwareInterface>hardware_interface/EffortJointInterface</hardwareInterface>
-      		<mechanicalReduction>1</mechanicalReduction>
-     	</actuator>
-  	</transmission>-->
-<xacro:property name="camera_link" value="0.1" /> <!-- Size of square 'camera' box -->
-	<joint name="camera_joint" type="fixed">
-    	<axis xyz="0 1 0" />
-    	<origin xyz="0.25 0.4 0.25" rpy="0 0 1.71"/>
-    	<parent link="wheel4"/>
-    	<child link="camera_link"/>
-  	</joint>
-  	<!-- Camera -->
-  	<link name="camera_link">
-    	<collision>
-      		<origin xyz="0 0 0" rpy="0 0 0"/>
-      		<geometry>
-    			<box size="${camera_link} ${camera_link} ${camera_link}"/>
-      		</geometry>
-    	</collision>
-		<visual>
-      		<origin xyz="0 0 0" rpy="0 0 0"/>
-      		<geometry>
-    			<box size="${camera_link} ${camera_link} ${camera_link}"/>
-      		</geometry>
-      		<material name="red"/>
-    	</visual>
-    	<inertial>
-      		<mass value="1e-5" />
-      		<origin xyz="0 0 0" rpy="0 0 0"/>
-      		<inertia ixx="1e-6" ixy="0" ixz="0" iyy="1e-6" iyz="0" izz="1e-6" />
-    	</inertial>
-  	</link>
 <xacro:link_leg name_leg = "first_leg" number_wheel = "wheel1"
 	            coord_joint = "1 1 0" angles_joint = "0 0 0"/>
@@ -180,43 +142,3 @@
   </plugin>
 </gazebo>
-<!-- camera -->
-  <gazebo reference="camera_link">
-    <sensor type="camera" name="camera1">
-      <update_rate>30.0</update_rate>
-      <camera name="head">
-        <horizontal_fov>1.3962634</horizontal_fov>
-        <image>
-          <width>800</width>
-          <height>800</height>
-          <format>R8G8B8</format>
-        </image>
-        <clip>
-          <near>0.02</near>
-          <far>300</far>
-        </clip>
-        <noise>
-          <type>gaussian</type>
-          <!-- Noise is sampled independently per pixel on each frame.
-               That pixel's noise value is added to each of its color
-               channels, which at that point lie in the range [0,1]. -->
-          <mean>0.0</mean>
-          <stddev>0.007</stddev>
-        </noise>
-      </camera>
-      <plugin name="camera_controller" filename="libgazebo_ros_camera.so">
-        <alwaysOn>true</alwaysOn>
-        <updateRate>0.0</updateRate>
-        <cameraName>camrobot/camera1</cameraName>
-        <imageTopicName>image_raw</imageTopicName>
-        <cameraInfoTopicName>camera_info</cameraInfoTopicName>
-        <frameName>camera_link</frameName>
-        <hackBaseline>0.07</hackBaseline>
-        <distortionK1>0.0</distortionK1>
-        <distortionK2>0.0</distortionK2>
-        <distortionK3>0.0</distortionK3>
-        <distortionT1>0.0</distortionT1>
-        <distortionT2>0.0</distortionT2>
-      </plugin>
-    </sensor>
-  </gazebo>
 </robot>
